Commit message: Make the lightsaber longer

File: ros2_ws/src/ur5_dynamics/urdf/ur5_with_tool.urdf.xacro (robot description, xacro)
@@ -6,7 +6,7 @@
   <link name="custom_tool">
     <visual>
-      <origin xyz="0 0 0.1" rpy="0 0 0"/>
+      <origin xyz="0 0 0.3" rpy="0 0 0"/>
       <geometry>
-        <cylinder radius="0.02" length="0.2"/>
+        <cylinder radius="0.02" length="0.6"/>
       </geometry>
       <material name="red">
